Commit message: 修复

File: source/robot_lab/data/Robots/atdog/dog_arm/urdf/dog_arm.urdf (robot description, URDF)
Before this commit: robot dog, 17 links, 16 joints
Links:
- link FL_calf: geometry collision mesh filename=package://dog_arm/meshes/left_front3.STL; visual mesh filename=package://dog_arm/meshes/left_front3.STL
- link FL_foot: geometry collision mesh filename=package://dog_arm/meshes/left_front4.STL; visual mesh filename=package://dog_arm/meshes/left_front4.STL
- link FL_hip: geometry collision mesh filename=package://dog_arm/meshes/left_front1.STL; visual mesh filename=package://dog_arm/meshes/left_front1.STL
- link FL_thigh: geometry collision mesh filename=package://dog_arm/meshes/left_front2.STL; visual mesh filename=package://dog_arm/meshes/left_front2.STL
- link FR_calf: geometry collision mesh filename=package://dog_arm/meshes/right_front3.STL; visual mesh filename=package://dog_arm/meshes/right_front3.STL
- link FR_foot: geometry collision mesh filename=package://dog_arm/meshes/right_front4.STL; visual mesh filename=package://dog_arm/meshes/right_front4.STL
- link FR_hip: geometry collision mesh filename=package://dog_arm/meshes/right_front1.STL; visual mesh filename=package://dog_arm/meshes/right_front1.STL
- link FR_thigh: geometry collision mesh filename=package://dog_arm/meshes/right_front2.STL; visual mesh filename=package://dog_arm/meshes/right_front2.STL
- link RL_calf: geometry collision mesh filename=package://dog_arm/meshes/left_behind3.STL; visual mesh filename=package://dog_arm/meshes/left_behind3.STL
- link RL_foot: geometry collision mesh filename=package://dog_arm/meshes/left_behind4.STL; visual mesh filename=package://dog_arm/meshes/left_behind4.STL
- link RL_hip: geometry collision mesh filename=package://dog_arm/meshes/left_behind1.STL; visual mesh filename=package://dog_arm/meshes/package://dog/meshes/left_behind1.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
- link RL_thigh: geometry collision mesh filename=package://dog_arm/meshes/left_behind2.STL; visual mesh filename=package://dog_arm/meshes/left_behind2.STL
- link RR_calf: geometry collision mesh filename=package://dog_arm/meshes/right_behind3.STL; visual mesh filename=package://dog_arm/meshes/right_behind3.STL
- link RR_foot: geometry collision mesh filename=package://dog_arm/meshes/right_behind4.STL; visual mesh filename=package://dog_arm/meshes/right_behind4.STL
- link RR_hip: geometry collision mesh filename=package://dog_arm/meshes/right_behind1.STL; visual mesh filename=package://dog_arm/meshes/right_behind1.STL
- link RR_thigh: geometry collision mesh filename=package://dog_arm/meshes/right_behind2.STL; visual mesh filename=package://dog_arm/meshes/right_behind2.STL
- link base_link: geometry collision mesh filename=package://dog_arm/meshes/base_link.STL; visual mesh filename=package://dog_arm/meshes/base_link.STL

Commit message: 修复

File: source/robot_lab/data/Robots/atdog/dog_arm/urdf/dog_arm.urdf (robot description, URDF)
Before this commit: robot dog, 17 links, 16 joints
Links:
- link RL_hip: geometry collision mesh filename=package://dog_arm/meshes/left_behind1.STL; visual mesh filename=package://dog_arm/meshes/left_behind1.STL

Commit message: 修复尝试

File: source/robot_lab/data/Robots/atdog/dog_arm/urdf/dog_arm.urdf (robot description, URDF)
Before this commit: robot dog, 17 links, 16 joints
Joints:
- joint FR_foot_joint: axis 0 0 -1 -> 0 0 1
- joint RR_foot_joint: axis 0 0 -1 -> 0 0 1

Commit message: 修复urdf

File: source/robot_lab/data/Robots/atdog/dog_arm/urdf/dog_arm.urdf (robot description, URDF)
Before this commit: robot dog, 17 links, 16 joints
Joints:
- joint FL_hip_joint: origin xyz=-0.0699998874435837 0.198599999999996 0.0620002717327733 rpy=1.5707963267949 0 -3.14159265358979 -> xyz=0.198599999999996 0.0699998874435837 0.0620002717327733 rpy=1.5707963267949 0 1.5707963267949
- joint FR_hip_joint: origin xyz=0.0700000000000028 0.198599999999997 0.0619999999999996 rpy=-1.5707963267949 0 0 -> xyz=0.198599999999997 -0.0700000000000028 0.0619999999999996 rpy=-1.5707963267949 0 -1.5707963267949
- joint RL_hip_joint: origin xyz=-0.0699999999999919 -0.198600000000003 0.0620000000000065 rpy=-1.57079632679489 0 3.14159265358979 -> xyz=-0.198600000000003 0.0699999999999919 0.0620000000000065 rpy=-1.57079632679489 0 1.5707963267949
- joint RR_hip_joint: origin xyz=0.0700000000000045 -0.1986 0.0620000000000064 rpy=1.57079632679489 0 0 -> xyz=-0.1986 -0.0700000000000045 0.0620000000000064 rpy=1.57079632679489 0 -1.5707963267949
