Commit message: 修改命名规范

File: source/robot_lab/data/Robots/atdog/dog/urdf/dog.urdf (robot description, URDF)
Before this commit: robot dog, 17 links, 16 joints
Links:
- removed link base_link
- removed link lb_link1
- removed link lb_link2
- removed link lb_link3
- removed link lf_link1
- removed link lf_link2
- removed link lf_link3
- removed link rb_link1
- removed link rb_link2
- removed link rb_link3
- removed link rf_link1
- removed link rf_link2
- removed link rf_link3
- added link FL_calf, mass  0.176947; collision mesh filename=package://dog/meshes/lf_link3.stl; visual mesh filename=package://dog/meshes/lf_link3.stl
- added link FL_hip, mass  0.648695; collision mesh filename=package://dog/meshes/lf_link1.stl; visual mesh filename=package://dog/meshes/lf_link1.stl
- added link FL_thigh, mass  1.076406; collision mesh filename=package://dog/meshes/lf_link2.stl; visual mesh filename=package://dog/meshes/lf_link2.stl
- added link FR_calf, mass 0.171842123814683; collision mesh filename=package://dog/meshes/rf_link3.stl; visual mesh filename=package://dog/meshes/rf_link3.stl
- added link FR_hip, mass 0.648695; collision mesh filename=package://dog/meshes/rf_link1.stl; visual mesh filename=package://dog/meshes/rf_link1.stl
- added link FR_thigh, mass 1.109062; collision mesh filename=package://dog/meshes/rf_link2.stl; visual mesh filename=package://dog/meshes/rf_link2.stl
- added link RL_calf, mass 0.171842123814683; collision mesh filename=package://dog/meshes/lb_link3.stl; visual mesh filename=package://dog/meshes/lb_link3.stl
- added link RL_hip, mass 0.648695; collision mesh filename=package://dog/meshes/lb_link1.stl; visual mesh filename=package://dog/meshes/lb_link1.stl
- added link RL_thigh, mass 1.105348; collision mesh filename=package://dog/meshes/lb_link2.stl; visual mesh filename=package://dog/meshes/lb_link2.stl
- added link RR_calf, mass 0.171842123814683; collision mesh filename=package://dog/meshes/rb_link3.stl; visual mesh filename=package://dog/meshes/rb_link3.stl
- added link RR_hip, mass  0.648695; collision mesh filename=package://dog/meshes/rb_link1.stl; visual mesh filename=package://dog/meshes/rb_link1.stl
- added link RR_thigh, mass 1.109062; collision mesh filename=package://dog/meshes/rb_link2.stl; visual mesh filename=package://dog/meshes/rb_link2.stl
- added link base, mass  5.073784; collision mesh filename=package://dog/meshes/base_link.stl; visual mesh filename=package://dog/meshes/base_link.stl
Joints:
- joint FL_calf_joint: child lf_link3 -> FL_calf; parent lf_link2 -> FL_thigh
- joint FL_foot_joint: parent lf_link3 -> FL_calf
- joint FL_hip_joint: child lf_link1 -> FL_hip; parent base_link -> base
- joint FL_thigh_joint: child lf_link2 -> FL_thigh; parent lf_link1 -> FL_hip
- joint FR_calf_joint: child rf_link3 -> FR_calf; parent rf_link2 -> FR_thigh
- joint FR_foot_joint: parent rf_link3 -> FR_calf
- joint FR_hip_joint: child rf_link1 -> FR_hip; parent base_link -> base
- joint FR_thigh_joint: child rf_link2 -> FR_thigh; parent rf_link1 -> FR_hip
- joint RL_calf_joint: child lb_link3 -> RL_calf; parent lb_link2 -> RL_thigh
- joint RL_foot_joint: parent lb_link3 -> RL_calf
- joint RL_hip_joint: child lb_link1 -> RL_hip; parent base_link -> base
- joint RL_thigh_joint: child lb_link2 -> RL_thigh; parent lb_link1 -> RL_hip
- joint RR_calf_joint: child rb_link3 -> RR_calf; parent rb_link2 -> RR_thigh
- joint RR_foot_joint: parent rb_link3 -> RR_calf
- joint RR_hip_joint: child rb_link1 -> RR_hip; parent base_link -> base
- joint RR_thigh_joint: child rb_link2 -> RR_thigh; parent rb_link1 -> RR_hip

File: source/robot_lab/data/Robots/atdog/dog2/urdf/dog2.urdf (robot description, URDF)
Before this commit: robot dog2, 17 links, 16 joints
Links:
- removed link body_link
- removed link lb_link1
- removed link lb_link2
- removed link lb_link3
- removed link lb_link4
- removed link lf_link1
- removed link lf_link2
- removed link lf_link3
- removed link lf_link4
- removed link rb_link1
- removed link rb_link2
- removed link rb_link3
- removed link rb_link4
- removed link rf_link1
- removed link rf_link2
- removed link rf_link3
- removed link rf_link4
- added link FL_calf, mass 0.466427846899075; collision mesh filename=package://dog2/meshes/lf_link3.stl; visual mesh filename=package://dog2/meshes/lf_link3.stl
- added link FL_foot, mass 0.084832216985374; collision mesh filename=package://dog2/meshes/lf_link4.stl; visual mesh filename=package://dog2/meshes/lf_link4.stl
- added link FL_hip, mass 0.676831582353488; collision mesh filename=package://dog2/meshes/lf_link1.stl; visual mesh filename=package://dog2/meshes/lf_link1.stl
- added link FL_thigh, mass 1.40828092509435; collision mesh filename=package://dog2/meshes/lf_link2.stl; visual mesh filename=package://dog2/meshes/lf_link2.stl
- added link FR_calf, mass 0.466427846899075; collision mesh filename=package://dog2/meshes/rf_link3.stl; visual mesh filename=package://dog2/meshes/rf_link3.stl
- added link FR_foot, mass 0.0848322169853742; collision mesh filename=package://dog2/meshes/rf_link4.stl; visual mesh filename=package://dog2/meshes/rf_link4.stl
- added link FR_hip, mass 0.677615723872956; collision mesh filename=package://dog2/meshes/rf_link1.stl; visual mesh filename=package://dog2/meshes/rf_link1.stl
- added link FR_thigh, mass 1.35333898941377; collision mesh filename=package://dog2/meshes/rf_link2.stl; visual mesh filename=package://dog2/meshes/rf_link2.stl
- added link RL_calf, mass 0.466427846899075; collision mesh filename=package://dog2/meshes/lb_link3.stl; visual mesh filename=package://dog2/meshes/lb_link3.stl
- added link RL_foot, mass 0.084832216985374; collision mesh filename=package://dog2/meshes/lb_link4.stl; visual mesh filename=package://dog2/meshes/lb_link4.stl
- added link RL_hip, mass 0.676831591069983; collision mesh filename=package://dog2/meshes/lb_link1.stl; visual mesh filename=package://dog2/meshes/lb_link1.stl
- added link RL_thigh, mass 1.40828094682296; collision mesh filename=package://dog2/meshes/lb_link2.stl; visual mesh filename=package://dog2/meshes/lb_link2.stl
- added link RR_calf, mass 0.456660190803704; collision mesh filename=package://dog2/meshes/rb_link3.stl; visual mesh filename=package://dog2/meshes/rb_link3.stl
- added link RR_foot, mass 0.084832216985374; collision mesh filename=package://dog2/meshes/rb_link4.stl; visual mesh filename=package://dog2/meshes/rb_link4.stl
- added link RR_hip, mass 0.676831591069986; collision mesh filename=package://dog2/meshes/rb_link1.stl; visual mesh filename=package://dog2/meshes/rb_link1.stl
- added link RR_thigh, mass 1.35333899025955; collision mesh filename=package://dog2/meshes/rb_link2.stl; visual mesh filename=package://dog2/meshes/rb_link2.stl
- added link base, mass 4.829; collision mesh filename=package://dog2/meshes/body_link.stl; visual mesh filename=package://dog2/meshes/body_link.stl
Joints:
- joint FL_calf_joint: child lf_link3 -> FL_calf; parent lf_link2 -> FL_thigh
- joint FL_foot_joint: child lf_link4 -> FL_foot; parent lf_link3 -> FL_calf
- joint FL_hip_joint: child lf_link1 -> FL_hip; parent body_link -> base
- joint FL_thigh_joint: child lf_link2 -> FL_thigh; parent lf_link1 -> FL_hip
- joint FR_calf_joint: child rf_link3 -> FR_calf; parent rf_link2 -> FR_thigh
- joint FR_foot_joint: child rf_link4 -> FR_foot; parent rf_link3 -> FR_calf
- joint FR_hip_joint: child rf_link1 -> FR_hip; parent body_link -> base
- joint FR_thigh_joint: child rf_link2 -> FR_thigh; parent rf_link1 -> FR_hip
- joint RL_calf_joint: child lb_link3 -> RL_calf; parent lb_link2 -> RL_thigh
- joint RL_foot_joint: child lb_link4 -> RL_foot; parent lb_link3 -> RL_calf
- joint RL_hip_joint: child lb_link1 -> RL_hip; parent body_link -> base
- joint RL_thigh_joint: child lb_link2 -> RL_thigh; parent lb_link1 -> RL_hip
- joint RR_calf_joint: child rb_link3 -> RR_calf; parent rb_link2 -> RR_thigh
- joint RR_foot_joint: child rb_link4 -> RR_foot; parent rb_link3 -> RR_calf
- joint RR_hip_joint: child rb_link1 -> RR_hip; parent body_link -> base
- joint RR_thigh_joint: child rb_link2 -> RR_thigh; parent rb_link1 -> RR_hip

Commit message: 微调URDF

File: source/robot_lab/data/Robots/atdog/dog/urdf/dog.urdf (robot description, URDF)
Before this commit: robot dog, 17 links, 16 joints
Links:
- removed link base
- added link base_link, mass  5.073784; collision mesh filename=package://dog/meshes/base_link.stl; visual mesh filename=package://dog/meshes/base_link.stl
Joints:
- joint FL_calf_joint: origin xyz=0.23001 0 0.0925 rpy=0 0 -1.6653 -> xyz=0.23001 0 0.0925 rpy=0 0 -1.5708
- joint FL_hip_joint: parent base -> base_link
- joint FR_calf_joint: origin xyz=0.22999 0 -0.0925 rpy=3.1416 0 -1.6804 -> xyz=0.22999 0 -0.0925 rpy=3.1416 0 -1.5708
- joint FR_hip_joint: parent base -> base_link
- joint RL_calf_joint: origin xyz=0.23001 0 0.0925 rpy=0 0 -1.629 -> xyz=0.23001 0 0.0925 rpy=0 0 -1.5708
- joint RL_hip_joint: parent base -> base_link
- joint RR_calf_joint: origin xyz=0.22999 0 0.0925 rpy=0 0 1.546 -> xyz=0.22999 0 0.0925 rpy=0 0 1.5708
- joint RR_hip_joint: parent base -> base_link

File: source/robot_lab/data/Robots/atdog/dog2/urdf/dog2.urdf (robot description, URDF)
Before this commit: robot dog2, 17 links, 16 joints
Joints:
- joint FL_thigh_joint: origin xyz=0.031298 0.00022929 0.06 rpy=-1.5708 0 -1.5639 -> xyz=0.031298 0.00022929 0.06 rpy=-1.5708 0 -1.5708
- joint FR_calf_joint: origin xyz=0.20707 -0.0041231 0.0726 rpy=0 0 1.5658 -> xyz=0.20707 -0.0041231 0.0726 rpy=0 0 1.5708
- joint FR_thigh_joint: origin xyz=-0.0313 -0.00018614 0.06 rpy=1.5708 0 -1.5644 -> xyz=-0.0313 -0.00018614 0.06 rpy=1.5708 0 -1.5708

Commit message: dog模型

File: source/robot_lab/data/Robots/atdog/dog/urdf/dog.urdf (robot description, URDF)
Before this commit: robot dog, 17 links, 16 joints
Links:
- link FL_calf: mass  0.176947 -> 0.240668495671817; geometry collision mesh filename=package://dog/meshes/left_front3.STL; visual mesh filename=package://dog/meshes/left_front3.STL
- link FL_foot: mass 0.432624 -> 0.432627569922019; geometry collision mesh filename=package://dog/meshes/left_front_whell.STL; visual mesh filename=package://dog/meshes/left_front_whell.STL
- link FL_hip: mass  0.648695 -> 0.638663512631356; geometry collision mesh filename=package://dog/meshes/left_front1.STL; visual mesh filename=package://dog/meshes/left_front1.STL
- link FL_thigh: mass  1.076406 -> 1.03305162619747; geometry collision mesh filename=package://dog/meshes/left_front2.STL; visual mesh filename=package://dog/meshes/left_front2.STL
- link FR_calf: mass 0.171842123814683 -> 0.240668495671817; geometry collision mesh filename=package://dog/meshes/right_front3.STL; visual mesh filename=package://dog/meshes/right_front3.STL
- link FR_foot: mass 0.432627569922016 -> 0.432306980666616; geometry collision mesh filename=package://dog/meshes/right_front_whell.STL; visual mesh filename=package://dog/meshes/right_front_whell.STL
- link FR_hip: mass 0.648695 -> 0.638663512631362; geometry collision mesh filename=package://dog/meshes/right_front1.STL; visual mesh filename=package://dog/meshes/right_front1.STL
- link FR_thigh: mass 1.109062 -> 1.03281470574407; geometry collision mesh filename=package://dog/meshes/right_front2.STL; visual mesh filename=package://dog/meshes/right_front2.STL
- link RL_calf: mass 0.171842123814683 -> 0.204986388414105; geometry collision mesh filename=package://dog/meshes/left_back3.STL; visual mesh filename=package://dog/meshes/left_back3.STL
- link RL_foot: mass 0.432627569922007 -> 0.432627569922008; geometry collision mesh filename=package://dog/meshes/right_back_whell.STL; visual mesh filename=package://dog/meshes/right_back_whell.STL
- link RL_hip: mass 0.648695 -> 0.638663512631339; geometry collision mesh filename=package://dog/meshes/left_back1.STL; visual mesh filename=package://dog/meshes/left_back1.STL
- link RL_thigh: mass 1.105348 -> 1.03179497617766; geometry collision mesh filename=package://dog/meshes/left_back2.STL; visual mesh filename=package://dog/meshes/left_back2.STL
- link RR_calf: mass 0.171842123814683 -> 0.240668495671816; geometry collision mesh filename=package://dog/meshes/right_back3.STL; visual mesh filename=package://dog/meshes/right_back3.STL
- link RR_foot: mass 0.432627569922011 -> 0.432627569922008; geometry collision mesh filename=package://dog/meshes/right_back_whell.STL; visual mesh filename=package://dog/meshes/right_back_whell.STL
- link RR_hip: mass  0.648695 -> 0.638663512641848; geometry collision mesh filename=package://dog/meshes/right_back_1.STL; visual mesh filename=package://dog/meshes/right_back_1.STL
- link RR_thigh: mass 1.109062 -> 1.03458097808249; geometry collision mesh filename=package://dog/meshes/right_back2.STL; visual mesh filename=package://dog/meshes/right_back2.STL
- link base_link: mass  5.073784 -> 4.4094; geometry collision mesh filename=package://dog/meshes/base_link.STL; visual mesh filename=package://dog/meshes/base_link.STL
Joints:
- joint FL_calf_joint: origin xyz=0.23001 0 0.0925 rpy=0 0 -1.5708 -> xyz=0.22969 -0.0028683 0.077109 rpy=0 0 -1.5708
- joint FL_foot_joint: axis 0 0 -1 -> 0 0 1; origin xyz=0.225 0 -0.0225 rpy=-3.1416 0 0 -> xyz=0.22212 0 0.049891 rpy=0 0 0
- joint FL_hip_joint: origin xyz=0.1916 0.069987 0.061999 rpy=0 1.5708 0 -> xyz=0.1986 0.07 0.06 rpy=1.5708 0 1.5708
- joint FL_thigh_joint: origin xyz=0 0.029313 0.060013 rpy=-1.5708 0 0 -> xyz=0.0313 0 0.053 rpy=-1.5708 0 -1.5708
- joint FR_calf_joint: origin xyz=0.22999 0 -0.0925 rpy=3.1416 0 -1.5708 -> xyz=0.22957 0.0028528 0.077109 rpy=0 0 1.5708
- joint FR_foot_joint: origin xyz=0.225 0 -0.0225 rpy=0 0 0 -> xyz=0.22212 0 0.047391 rpy=0 0 0
- joint FR_hip_joint: origin xyz=0.1916 -0.070013 0.061999 rpy=0 1.5708 0 -> xyz=0.1986 -0.07 0.06 rpy=-1.5708 0 -1.5708
- joint FR_thigh_joint: axis 0 0 -1 -> 0 0 1; origin xyz=0 -0.029287 0.059987 rpy=-1.5708 0 0 -> xyz=0.0313 0 0.053 rpy=1.5708 0 1.5708
- joint RL_calf_joint: origin xyz=0.23001 0 0.0925 rpy=0 0 -1.5708 -> xyz=0.22983 -0.0028798 0.077109 rpy=0 0 -1.5708
- joint RL_foot_joint: origin xyz=0.225 0 -0.0225 rpy=0 0 0 -> xyz=0.22212 0 0.047391 rpy=0 0 0
- joint RL_hip_joint: origin xyz=-0.1916 0.070013 0.061999 rpy=3.1416 1.5708 0 -> xyz=-0.1986 0.07 0.06 rpy=-1.5708 0 1.5708
- joint RL_thigh_joint: origin xyz=0 -0.029287 0.059987 rpy=1.5708 0 0 -> xyz=0.0313 0 0.053 rpy=1.5708 0 1.5708
- joint RR_calf_joint: origin xyz=0.22999 0 0.0925 rpy=0 0 1.5708 -> xyz=0.22977 0.0028755 0.077109 rpy=0 0 1.5708
- joint RR_foot_joint: origin xyz=0.225 0 -0.0225 rpy=0 0 0 -> xyz=0.22212 0 0.047391 rpy=0 0 0
- joint RR_hip_joint: origin xyz=-0.1916 -0.069987 0.061999 rpy=3.1416 1.5708 0 -> xyz=-0.1986 -0.07 0.06 rpy=1.5708 0 -1.5708
- joint RR_thigh_joint: origin xyz=0 0.029313 0.060013 rpy=-1.5708 0 0 -> xyz=0.0313 0 0.053 rpy=-1.5708 0 -1.5708

Commit message: 更新轮足狗ATDog的URDF

File: source/robot_lab/data/Robots/atdog/dog/urdf/dog.urdf (robot description, URDF)
Before this commit: robot dog, 17 links, 16 joints
Links:
- link FL_calf: mass 0.240668495671817 -> 0.239198906199937; geometry collision mesh filename=package://dog/meshes/left_front3.stl; visual mesh filename=package://dog/meshes/left_front3.stl
- link FL_foot: mass 0.432627569922019 -> 0.759852059316646; geometry collision mesh filename=package://dog/meshes/left_front4.stl; visual mesh filename=package://dog/meshes/left_front4.stl
- link FL_hip: mass 0.638663512631356 -> 0.742829095910112; geometry collision mesh filename=package://dog/meshes/left_front1.stl; visual mesh filename=package://dog/meshes/left_front1.stl
- link FL_thigh: mass 1.03305162619747 -> 1.18835534771936; geometry collision mesh filename=package://dog/meshes/left_front2.stl; visual mesh filename=package://dog/meshes/left_front2.stl
- link FR_calf: mass 0.240668495671817 -> 0.236883938830138; geometry collision mesh filename=package://dog/meshes/right_front3.stl; visual mesh filename=package://dog/meshes/right_front3.stl
- link FR_foot: mass 0.432306980666616 -> 0.75985; geometry collision mesh filename=package://dog/meshes/right_front4.stl; visual mesh filename=package://dog/meshes/right_front4.stl
- link FR_hip: mass 0.638663512631362 -> 0.742829095911341; geometry collision mesh filename=package://dog/meshes/right_front1.stl; visual mesh filename=package://dog/meshes/right_front1.stl
- link FR_thigh: mass 1.03281470574407 -> 1.19692172233053; geometry collision mesh filename=package://dog/meshes/right_front2.stl; visual mesh filename=package://dog/meshes/right_front2.stl
- link RL_calf: mass 0.204986388414105 -> 0.239198906199937; geometry collision mesh filename=package://dog/meshes/left_behind3.stl; visual mesh filename=package://dog/meshes/left_behind3.stl
- link RL_foot: mass 0.432627569922008 -> 0.759852059316647; geometry collision mesh filename=package://dog/meshes/left_behind4.stl; visual mesh filename=package://dog/meshes/left_behind4.stl
- link RL_hip: mass 0.638663512631339 -> 0.742829095909968; geometry collision mesh filename=package://dog/meshes/left_behind1.stl; visual mesh filename=package://dog/meshes/left_behind1.stl
- link RL_thigh: mass 1.03179497617766 -> 1.18835557567372; geometry collision mesh filename=package://dog/meshes/left_behind2.stl; visual mesh filename=package://dog/meshes/left_behind2.stl
- link RR_calf: mass 0.240668495671816 -> 0.239198906199937; geometry collision mesh filename=package://dog/meshes/right_behind3.stl; visual mesh filename=package://dog/meshes/right_behind3.stl
- link RR_foot: mass 0.432627569922008 -> 0.759852059316651; geometry collision mesh filename=package://dog/meshes/right_behind4.stl; visual mesh filename=package://dog/meshes/right_behind4.stl
- link RR_hip: mass 0.638663512641848 -> 0.742829095909967; geometry collision mesh filename=package://dog/meshes/right_behind1.stl; visual mesh filename=package://dog/meshes/right_behind1.stl
- link RR_thigh: mass 1.03458097808249 -> 1.19692196706229; geometry collision mesh filename=package://dog/meshes/right_behind2.stl; visual mesh filename=package://dog/meshes/right_behind2.stl
- link base_link: mass 4.4094 -> 5.21190024516352; geometry collision mesh filename=package://dog/meshes/base_link.stl; visual mesh filename=package://dog/meshes/base_link.stl
Joints:
- joint FL_calf_joint: limit lower=-3.14 upper=3.14 effort=23 velocity=30 -> lower=-3.1415926 upper=3.1415926 effort=40 velocity=20; origin xyz=0.22969 -0.0028683 0.077109 rpy=0 0 -1.5708 -> xyz=0.23 0 0.07975 rpy=0 0 -1.5704
- joint FL_foot_joint: limit effort=2 velocity=13 -> (none); origin xyz=0.22212 0 0.049891 rpy=0 0 0 -> xyz=0.225 0 -0.01125 rpy=0 0 0
- joint FL_hip_joint: limit lower=-3.14 upper=3.14 effort=23 velocity=30 -> lower=-3.1415926 upper=3.1415926 effort=23 velocity=30; origin xyz=0.1986 0.07 0.06 rpy=1.5708 0 1.5708 -> xyz=0.198599827436973 0.0699998874434311 0.0620002761469703 rpy=1.5707963267949 0 1.5707963267949
- joint FL_thigh_joint: limit lower=-3.14 upper=3.14 effort=23 velocity=30 -> lower=-3.1415926 upper=3.1415926 effort=23 velocity=30; origin xyz=0.0313 0 0.053 rpy=-1.5708 0 -1.5708 -> xyz=0.0358 0 0.053 rpy=-1.5708 0 -1.5708
- joint FR_calf_joint: limit lower=-3.14 upper=3.14 effort=23 velocity=30 -> lower=-3.1415926 upper=3.1415926 effort=40 velocity=20; origin xyz=0.22957 0.0028528 0.077109 rpy=0 0 1.5708 -> xyz=0.229999999999999 0 0.079749999999998 rpy=0 0 1.5704
- joint FR_foot_joint: limit effort=2 velocity=13 -> (none); origin xyz=0.22212 0 0.047391 rpy=0 0 0 -> xyz=0.225 0 -0.01125 rpy=0 0 0
- joint FR_hip_joint: limit lower=-3.14 upper=3.14 effort=23 velocity=30 -> lower=-3.1415926 upper=3.1415926 effort=23 velocity=30; origin xyz=0.1986 -0.07 0.06 rpy=-1.5708 0 -1.5708 -> xyz=0.198600112556418 -0.0700000000000034 0.0620005478797402 rpy=-1.5707963267949 0 -1.5707963267949
- joint FR_thigh_joint: limit lower=-3.14 upper=3.14 effort=23 velocity=30 -> lower=-3.1415926 upper=3.1415926 effort=23 velocity=30; origin xyz=0.0313 0 0.053 rpy=1.5708 0 1.5708 -> xyz=0.0357999999999982 0 0.052999887443579 rpy=1.57079632679493 0 1.5707963267949
- joint RL_calf_joint: limit lower=-3.14 upper=3.14 effort=23 velocity=30 -> lower=-3.1415926 upper=3.1415926 effort=40 velocity=20; origin xyz=0.22983 -0.0028798 0.077109 rpy=0 0 -1.5708 -> xyz=0.230000000092392 0 0.0797499999975051 rpy=0 0 -1.5704
- joint RL_foot_joint: limit effort=2 velocity=13 -> (none); origin xyz=0.22212 0 0.047391 rpy=0 0 0 -> xyz=0.225 0 -0.01125 rpy=0 0 0
- joint RL_hip_joint: limit lower=-3.14 upper=3.14 effort=23 velocity=30 -> lower=-3.1415926 upper=3.1415926 effort=23 velocity=30; origin xyz=-0.1986 0.07 0.06 rpy=-1.5708 0 1.5708 -> xyz=-0.198600000000003 0.0699999999999925 0.0620000000000055 rpy=-1.5707963267949 0 1.57079632679489
- joint RL_thigh_joint: limit lower=-3.14 upper=3.14 effort=23 velocity=30 -> lower=-3.1415926 upper=3.1415926 effort=23 velocity=30; origin xyz=0.0313 0 0.053 rpy=1.5708 0 1.5708 -> xyz=0.0358000000000075 0 0.0530000000000009 rpy=1.57079632679488 0 1.5707963267949
- joint RR_calf_joint: limit lower=-3.14 upper=3.14 effort=23 velocity=30 -> lower=-3.1415926 upper=3.1415926 effort=40 velocity=20; origin xyz=0.22977 0.0028755 0.077109 rpy=0 0 1.5708 -> xyz=0.230000000090279 0 0.0797499999999652 rpy=0 0 1.5704
- joint RR_foot_joint: limit effort=2 velocity=13 -> (none); origin xyz=0.22212 0 0.047391 rpy=0 0 0 -> xyz=0.225 0 -0.01125 rpy=0 0 0
- joint RR_hip_joint: limit lower=-3.14 upper=3.14 effort=23 velocity=30 -> lower=-3.1415926 upper=3.1415926 effort=23 velocity=30; origin xyz=-0.1986 -0.07 0.06 rpy=1.5708 0 -1.5708 -> xyz=-0.1986 -0.0700000000000039 0.0620000000000056 rpy=1.5707963267949 0 -1.5707963267949
- joint RR_thigh_joint: limit lower=-3.14 upper=3.14 effort=23 velocity=30 -> lower=-3.1415926 upper=3.1415926 effort=23 velocity=30; origin xyz=0.0313 0 0.053 rpy=-1.5708 0 -1.5708 -> xyz=0.0358 0 0.0530000000000005 rpy=-1.57079632679491 0 -1.5707963267949
