Commit message: 导入模型

File: source/robot_lab/data/Robots/atdog/dog2/urdf/dog2.urdf (robot description, URDF)
Before this commit: robot dog2, 17 links, 16 joints
Links:
- removed link FL_calf
- removed link FL_foot
- removed link FL_hip
- removed link FL_thigh
- removed link FR_calf
- removed link FR_foot
- removed link FR_hip
- removed link FR_thigh
- removed link RL_calf
- removed link RL_foot
- removed link RL_hip
- removed link RL_thigh
- removed link RR_calf
- removed link RR_foot
- removed link RR_hip
- removed link RR_thigh
- removed link base
- added link body_link, mass 2.6721; collision mesh filename=package://dog2/meshes/body_link.STL; visual mesh filename=package://dog2/meshes/body_link.STL
- added link lb_link1, mass 0.30939; collision mesh filename=package://dog2/meshes/lb_link1.STL; visual mesh filename=package://dog2/meshes/lb_link1.STL
- added link lb_link2, mass 0.779; collision mesh filename=package://dog2/meshes/lb_link2.STL; visual mesh filename=package://dog2/meshes/lb_link2.STL
- added link lb_link3, mass 0.57476; collision mesh filename=package://dog2/meshes/lb_link3.STL; visual mesh filename=package://dog2/meshes/lb_link3.STL
- added link lb_link4, mass 0.084832; collision mesh filename=package://dog2/meshes/lb_link4.STL; visual mesh filename=package://dog2/meshes/lb_link4.STL
- added link lf_link1, mass 0.30939; collision mesh filename=package://dog2/meshes/lf_link1.STL; visual mesh filename=package://dog2/meshes/lf_link1.STL
- added link lf_link2, mass 0.779; collision mesh filename=package://dog2/meshes/lf_link2.STL; visual mesh filename=package://dog2/meshes/lf_link2.STL
- added link lf_link3, mass 0.57476; collision mesh filename=package://dog2/meshes/lf_link3.STL; visual mesh filename=package://dog2/meshes/lf_link3.STL
- added link lf_link4, mass 0.084832; collision mesh filename=package://dog2/meshes/lf_link4.STL; visual mesh filename=package://dog2/meshes/lf_link4.STL
- added link rb_link1, mass 0; collision mesh filename=package://dog2/meshes/rb_link1.STL; visual mesh filename=package://dog2/meshes/rb_link1.STL
- added link rb_link2, mass 0.72406; collision mesh filename=package://dog2/meshes/rb_link2.STL; visual mesh filename=package://dog2/meshes/rb_link2.STL
- added link rb_link3, mass 0.56499; collision mesh filename=package://dog2/meshes/rb_link3.STL; visual mesh filename=package://dog2/meshes/rb_link3.STL
- added link rb_link4, mass 0.084832; collision mesh filename=package://dog2/meshes/rb_link4.STL; visual mesh filename=package://dog2/meshes/rb_link4.STL
- added link rf_link1, mass 0.30939; collision mesh filename=package://dog2/meshes/rf_link1.STL; visual mesh filename=package://dog2/meshes/rf_link1.STL
- added link rf_link2, mass 0.83975; collision mesh filename=package://dog2/meshes/rf_link2.STL; visual mesh filename=package://dog2/meshes/rf_link2.STL
- added link rf_link3, mass 0.57476; collision mesh filename=package://dog2/meshes/rf_link3.STL; visual mesh filename=package://dog2/meshes/rf_link3.STL
- added link rf_link4, mass 0.084832; collision mesh filename=package://dog2/meshes/rf_link4.STL; visual mesh filename=package://dog2/meshes/rf_link4.STL
Joints:
- removed joint FL_calf_joint
- removed joint FL_foot_joint
- removed joint FL_hip_joint
- removed joint FL_thigh_joint
- removed joint FR_calf_joint
- removed joint FR_foot_joint
- removed joint FR_hip_joint
- removed joint FR_thigh_joint
- removed joint RL_calf_joint
- removed joint RL_foot_joint
- removed joint RL_hip_joint
- removed joint RL_thigh_joint
- removed joint RR_calf_joint
- removed joint RR_foot_joint
- removed joint RR_hip_joint
- removed joint RR_thigh_joint
- added joint lb_joint1: type revolute, parent body_link, child lb_link1, origin xyz=-0.2098 0.058472 0.038542 rpy=-1.5708 0 1.5708, axis 0 0 1, limit lower=0 upper=0 effort=0 velocity=0
- added joint lb_joint2: type revolute, parent lb_link1, child lb_link2, origin xyz=0.031301 -1.3226E-05 0.091299 rpy=1.5708 0.72621 1.5708, axis 0 0 1, limit lower=0 upper=0 effort=0 velocity=0
- added joint lb_joint3: type revolute, parent lb_link2, child lb_link3, origin xyz=0.22785 -0.027525 0.0726 rpy=0 0 1.7983, axis 0 0 1, limit lower=0 upper=0 effort=0 velocity=0
- added joint lb_joint4: type continuous, parent lb_link3, child lb_link4, origin xyz=0.22 0 0 rpy=3.1416 0 -1.5708, axis 0 0 1
- added joint lf_joint1: type revolute, parent body_link, child lf_link1, origin xyz=0.1834 0.058474 0.038542 rpy=1.5708 0 1.5708, axis 0 0 1, limit lower=0 upper=0 effort=0 velocity=0
- added joint lf_joint2: type prismatic, parent lf_link1, child lf_link2, origin xyz=0.031298 0.00022929 0.06 rpy=-1.5708 0.60394 -1.5639, axis 0 0 1, limit lower=0 upper=0 effort=0 velocity=0
- added joint lf_joint3: type revolute, parent lf_link2, child lf_link3, origin xyz=0.20707 -0.0041231 0.0716 rpy=0 0 -1.5104, axis 0 0 1, limit lower=0 upper=0 effort=0 velocity=0
- added joint lf_joint4: type fixed, parent lf_link3, child lf_link4, origin xyz=0.22 0 0.001 rpy=0 0 -1.5708, axis 0 0 0
- added joint rb_joint1: type revolute, parent body_link, child rb_link1, origin xyz=-0.2098 -0.061526 0.038569 rpy=-1.5708 0 1.5708, axis 0 0 1, limit lower=0 upper=0 effort=0 velocity=0
- added joint rb_joint2: type revolute, parent rb_link1, child rb_link2, origin xyz=-0.031301 1.3226E-05 0.091299 rpy=-1.5708 0.68838 1.5708, axis 0 0 1, limit lower=0 upper=0 effort=0 velocity=0
- added joint rb_joint3: type revolute, parent rb_link2, child rb_link3, origin xyz=0.22695 0.028294 0.0726 rpy=0 0 -1.7533, axis 0 0 1, limit lower=0 upper=0 effort=0 velocity=0
- added joint rb_joint4: type fixed, parent rb_link3, child rb_link4, origin xyz=0.22 0 0 rpy=3.1416 0 -1.5708, axis 0 0 0
- added joint rf_joint1: type revolute, parent body_link, child rf_link1, origin xyz=0.1834 -0.061526 0.038542 rpy=1.5708 0 1.5708, axis 0 0 1, limit lower=0 upper=0 effort=0 velocity=0
- added joint rf_joint2: type revolute, parent rf_link1, child rf_link2, origin xyz=-0.0313 -0.00018614 0.06 rpy=1.5708 0.63691 -1.5644, axis 0 0 1, limit lower=0 upper=0 effort=0 velocity=0
- added joint rf_joint3: type revolute, parent rf_link2, child rf_link3, origin xyz=0.20707 -0.0041231 0.0726 rpy=0 0 1.5658, axis 0 0 1, limit lower=0 upper=0 effort=0 velocity=0
- added joint rf_joint4: type fixed, parent rf_link3, child rf_link4, origin xyz=0.22 0 0 rpy=-3.1416 0 -1.5708, axis 0 0 0

Commit message: 1

File: source/robot_lab/data/Robots/atdog/dog2/urdf/dog2.urdf (robot description, URDF)
Before this commit: robot dog2, 17 links, 16 joints
Links:
- removed link body_link
- removed link lb_link1
- removed link lb_link2
- removed link lb_link3
- removed link lb_link4
- removed link lf_link1
- removed link lf_link2
- removed link lf_link3
- removed link lf_link4
- removed link rb_link1
- removed link rb_link2
- removed link rb_link3
- removed link rb_link4
- removed link rf_link1
- removed link rf_link2
- removed link rf_link3
- removed link rf_link4
- added link FL_calf, mass 0.57476; collision mesh filename=package://dog2/meshes/lf_link3.STL; visual mesh filename=package://dog2/meshes/lf_link3.STL
- added link FL_foot, mass 0.084832; collision mesh filename=package://dog2/meshes/lf_link4.STL; visual mesh filename=package://dog2/meshes/lf_link4.STL
- added link FL_hip, mass 0.30939; collision mesh filename=package://dog2/meshes/lf_link1.STL; visual mesh filename=package://dog2/meshes/lf_link1.STL
- added link FL_thigh, mass 0.779; collision mesh filename=package://dog2/meshes/lf_link2.STL; visual mesh filename=package://dog2/meshes/lf_link2.STL
- added link FR_calf, mass 0.57476; collision mesh filename=package://dog2/meshes/rf_link3.STL; visual mesh filename=package://dog2/meshes/rf_link3.STL
- added link FR_foot, mass 0.084832; collision mesh filename=package://dog2/meshes/rf_link4.STL; visual mesh filename=package://dog2/meshes/rf_link4.STL
- added link FR_hip, mass 0.30939; collision mesh filename=package://dog2/meshes/rf_link1.STL; visual mesh filename=package://dog2/meshes/rf_link1.STL
- added link FR_thigh, mass 0.83975; collision mesh filename=package://dog2/meshes/rf_link2.STL; visual mesh filename=package://dog2/meshes/rf_link2.STL
- added link RL_calf, mass 0.57476; collision mesh filename=package://dog2/meshes/lb_link3.STL; visual mesh filename=package://dog2/meshes/lb_link3.STL
- added link RL_foot, mass 0.084832; collision mesh filename=package://dog2/meshes/lb_link4.STL; visual mesh filename=package://dog2/meshes/lb_link4.STL
- added link RL_hip, mass 0.30939; collision mesh filename=package://dog2/meshes/lb_link1.STL; visual mesh filename=package://dog2/meshes/lb_link1.STL
- added link RL_thigh, mass 0.779; collision mesh filename=package://dog2/meshes/lb_link2.STL; visual mesh filename=package://dog2/meshes/lb_link2.STL
- added link RR_calf, mass 0.56499; collision mesh filename=package://dog2/meshes/rb_link3.STL; visual mesh filename=package://dog2/meshes/rb_link3.STL
- added link RR_foot, mass 0.084832; collision mesh filename=package://dog2/meshes/rb_link4.STL; visual mesh filename=package://dog2/meshes/rb_link4.STL
- added link RR_hip, mass 0; collision mesh filename=package://dog2/meshes/rb_link1.STL; visual mesh filename=package://dog2/meshes/rb_link1.STL
- added link RR_thigh, mass 0.72406; collision mesh filename=package://dog2/meshes/rb_link2.STL; visual mesh filename=package://dog2/meshes/rb_link2.STL
- added link base, mass 2.6721; collision mesh filename=package://dog2/meshes/body_link.STL; visual mesh filename=package://dog2/meshes/body_link.STL
Joints:
- removed joint lb_joint1
- removed joint lb_joint2
- removed joint lb_joint3
- removed joint lb_joint4
- removed joint lf_joint1
- removed joint lf_joint2
- removed joint lf_joint3
- removed joint lf_joint4
- removed joint rb_joint1
- removed joint rb_joint2
- removed joint rb_joint3
- removed joint rb_joint4
- removed joint rf_joint1
- removed joint rf_joint2
- removed joint rf_joint3
- removed joint rf_joint4
- added joint FL_calf_joint: type revolute, parent FL_thigh, child FL_calf, origin xyz=0.20707 -0.0041231 0.0716 rpy=0 0 -1.5104, axis 0 0 1, limit lower=0 upper=0 effort=0 velocity=0
- added joint FL_foot_joint: type fixed, parent FL_calf, child FL_foot, origin xyz=0.22 0 0.001 rpy=0 0 -1.5708, axis 0 0 0
- added joint FL_hip_joint: type revolute, parent base, child FL_hip, origin xyz=0.1834 0.058474 0.038542 rpy=1.5708 0 1.5708, axis 0 0 1, limit lower=0 upper=0 effort=0 velocity=0
- added joint FL_thigh_joint: type prismatic, parent FL_hip, child FL_thigh, origin xyz=0.031298 0.00022929 0.06 rpy=-1.5708 0.60394 -1.5639, axis 0 0 1, limit lower=-1.0 upper=1.0 effort=20 velocity=20
- added joint FR_calf_joint: type revolute, parent FR_thigh, child FR_calf, origin xyz=0.20707 -0.0041231 0.0726 rpy=0 0 1.5658, axis 0 0 1, limit lower=0 upper=0 effort=0 velocity=0
- added joint FR_foot_joint: type fixed, parent FR_calf, child FR_foot, origin xyz=0.22 0 0 rpy=3.1416 0 -1.5708, axis 0 0 0
- added joint FR_hip_joint: type revolute, parent base, child FR_hip, origin xyz=0.1834 -0.061526 0.038542 rpy=1.5708 0 1.5708, axis 0 0 1, limit lower=0 upper=0 effort=0 velocity=0
- added joint FR_thigh_joint: type revolute, parent FR_hip, child FR_thigh, origin xyz=-0.0313 -0.00018614 0.06 rpy=1.5708 0.63691 -1.5644, axis 0 0 1, limit lower=-1.0 upper=1.0 effort=20 velocity=20
- added joint RL_calf_joint: type revolute, parent RL_thigh, child RL_calf, origin xyz=0.22785 -0.027525 0.0726 rpy=0 0 1.7983, axis 0 0 1, limit lower=0 upper=0 effort=0 velocity=0
- added joint RL_foot_joint: type fixed, parent RL_calf, child RL_foot, origin xyz=0.22 0 0 rpy=3.1416 0 -1.5708, axis 0 0 0
- added joint RL_hip_joint: type revolute, parent base, child RL_hip, origin xyz=-0.2098 0.058472 0.038542 rpy=-1.5708 0 1.5708, axis 0 0 1, limit lower=0 upper=0 effort=0 velocity=0
- added joint RL_thigh_joint: type revolute, parent RL_hip, child RL_thigh, origin xyz=0.031301 -1.3226E-05 0.091299 rpy=1.5708 0.72621 1.5708, axis 0 0 1, limit lower=-1.0 upper=1.0 effort=20 velocity=20
- added joint RR_calf_joint: type revolute, parent RR_thigh, child RR_calf, origin xyz=0.22695 0.028294 0.0726 rpy=0 0 -1.7533, axis 0 0 1, limit lower=0 upper=0 effort=0 velocity=0
- added joint RR_foot_joint: type fixed, parent RR_calf, child RR_foot, origin xyz=0.22 0 0 rpy=-3.1416 0 -1.5708, axis 0 0 0
- added joint RR_hip_joint: type revolute, parent base, child RR_hip, origin xyz=-0.2098 -0.061526 0.038569 rpy=-1.5708 0 1.5708, axis 0 0 1, limit lower=0 upper=0 effort=0 velocity=0
- added joint RR_thigh_joint: type revolute, parent RR_hip, child RR_thigh, origin xyz=-0.031301 1.3226E-05 0.091299 rpy=-1.5708 0.68838 1.5708, axis 0 0 1, limit lower=-1.0 upper=1.0 effort=20 velocity=20

Commit message: 更新机器人模型

File: source/robot_lab/data/Robots/atdog/dog2/urdf/dog2.urdf (robot description, URDF)
Before this commit: robot dog2, 17 links, 16 joints
Links:
- link body_link: mass 2.6721 -> 4.829; geometry collision mesh filename=package://dog2/meshes/body_link.stl; visual mesh filename=package://dog2/meshes/body_link.stl
- link lb_link1: mass 0.30939 -> 0.676831591069983; geometry collision mesh filename=package://dog2/meshes/lb_link1.stl; visual mesh filename=package://dog2/meshes/lb_link1.stl
- link lb_link2: mass 0.779 -> 1.40828094682296; geometry collision mesh filename=package://dog2/meshes/lb_link2.stl; visual mesh filename=package://dog2/meshes/lb_link2.stl
- link lb_link3: mass 0.57476 -> 0.466427846899075; geometry collision mesh filename=package://dog2/meshes/lb_link3.stl; visual mesh filename=package://dog2/meshes/lb_link3.stl
- link lb_link4: mass 0.084832 -> 0.084832216985374; geometry collision mesh filename=package://dog2/meshes/lb_link4.stl; visual mesh filename=package://dog2/meshes/lb_link4.stl
- link lf_link1: mass 0.30939 -> 0.676831582353488; geometry collision mesh filename=package://dog2/meshes/lf_link1.stl; visual mesh filename=package://dog2/meshes/lf_link1.stl
- link lf_link2: mass 0.779 -> 1.40828092509435; geometry collision mesh filename=package://dog2/meshes/lf_link2.stl; visual mesh filename=package://dog2/meshes/lf_link2.stl
- link lf_link3: mass 0.57476 -> 0.466427846899075; geometry collision mesh filename=package://dog2/meshes/lf_link3.stl; visual mesh filename=package://dog2/meshes/lf_link3.stl
- link lf_link4: mass 0.084832 -> 0.084832216985374; geometry collision mesh filename=package://dog2/meshes/lf_link4.stl; visual mesh filename=package://dog2/meshes/lf_link4.stl
- link rb_link1: mass 0 -> 0.676831591069986; geometry collision mesh filename=package://dog2/meshes/rb_link1.stl; visual mesh filename=package://dog2/meshes/rb_link1.stl
- link rb_link2: mass 0.72406 -> 1.35333899025955; geometry collision mesh filename=package://dog2/meshes/rb_link2.stl; visual mesh filename=package://dog2/meshes/rb_link2.stl
- link rb_link3: mass 0.56499 -> 0.456660190803704; geometry collision mesh filename=package://dog2/meshes/rb_link3.stl; visual mesh filename=package://dog2/meshes/rb_link3.stl
- link rb_link4: mass 0.084832 -> 0.084832216985374; geometry collision mesh filename=package://dog2/meshes/rb_link4.stl; visual mesh filename=package://dog2/meshes/rb_link4.stl
- link rf_link1: mass 0.30939 -> 0.677615723872956; geometry collision mesh filename=package://dog2/meshes/rf_link1.stl; visual mesh filename=package://dog2/meshes/rf_link1.stl
- link rf_link2: mass 0.83975 -> 1.35333898941377; geometry collision mesh filename=package://dog2/meshes/rf_link2.stl; visual mesh filename=package://dog2/meshes/rf_link2.stl
- link rf_link3: mass 0.57476 -> 0.466427846899075; geometry collision mesh filename=package://dog2/meshes/rf_link3.stl; visual mesh filename=package://dog2/meshes/rf_link3.stl
- link rf_link4: mass 0.084832 -> 0.0848322169853742; geometry collision mesh filename=package://dog2/meshes/rf_link4.stl; visual mesh filename=package://dog2/meshes/rf_link4.stl
Joints:
- removed joint lb_joint1
- removed joint lb_joint2
- removed joint lb_joint3
- removed joint lb_joint4
- removed joint lf_joint1
- removed joint lf_joint2
- removed joint lf_joint3
- removed joint lf_joint4
- removed joint rb_joint1
- removed joint rb_joint2
- removed joint rb_joint3
- removed joint rb_joint4
- removed joint rf_joint1
- removed joint rf_joint2
- removed joint rf_joint3
- removed joint rf_joint4
- added joint FL_calf_joint: type revolute, parent lf_link2, child lf_link3, origin xyz=0.20707 -0.0041231 0.0716 rpy=0 0 -1.570796, axis 0 0 1, limit lower=-3.14159 upper=3.14159 effort=23 velocity=30
- added joint FL_foot_joint: type fixed, parent lf_link3, child lf_link4, origin xyz=0.22 0 0.001 rpy=0 0 -1.5708, axis 0 0 0
- added joint FL_hip_joint: type revolute, parent body_link, child lf_link1, origin xyz=0.18433 0.058364 0.045534 rpy=1.5708 0 1.5708, axis 0 0 1, limit lower=-3.14159 upper=3.14159 effort=23 velocity=30
- added joint FL_thigh_joint: type revolute, parent lf_link1, child lf_link2, origin xyz=0.031298 0.00022929 0.06 rpy=-1.5708 0 -1.5639, axis 0 0 1, limit lower=-3.14159 upper=3.14159 effort=23 velocity=30
- added joint FR_calf_joint: type revolute, parent rf_link2, child rf_link3, origin xyz=0.20707 -0.0041231 0.0726 rpy=0 0 1.5658, axis 0 0 1, limit lower=-3.14159 upper=3.14159 effort=23 velocity=30
- added joint FR_foot_joint: type fixed, parent rf_link3, child rf_link4, origin xyz=0.22 0 0 rpy=3.1416 0 -1.5708, axis 0 0 0
- added joint FR_hip_joint: type revolute, parent body_link, child rf_link1, origin xyz=0.18643 -0.06136 0.03776 rpy=1.5708 0 1.5708, axis 0 0 1, limit lower=-3.14159 upper=3.14159 effort=23 velocity=30
- added joint FR_thigh_joint: type revolute, parent rf_link1, child rf_link2, origin xyz=-0.0313 -0.00018614 0.06 rpy=1.5708 0 -1.5644, axis 0 0 1, limit lower=-3.14159 upper=3.14159 effort=23 velocity=30
- added joint RL_calf_joint: type revolute, parent lb_link2, child lb_link3, origin xyz=0.20711 0 0.0746 rpy=0 0 -1.570796, axis 0 0 1, limit lower=-3.14159 upper=3.14159 effort=23 velocity=30
- added joint RL_foot_joint: type fixed, parent lb_link3, child lb_link4, origin xyz=0.22 0 0 rpy=3.1416 0 -1.5708, axis 0 0 0
- added joint RL_hip_joint: type revolute, parent body_link, child lb_link1, origin xyz=-0.20677 0.058639 0.03776 rpy=-1.5708 0 1.5708, axis 0 0 1, limit lower=-3.14159 upper=3.14159 effort=23 velocity=30
- added joint RL_thigh_joint: type revolute, parent lb_link1, child lb_link2, origin xyz=0.029301 -1.3226E-05 0.06 rpy=1.5708 0 1.5708, axis 0 0 1, limit lower=-3.14159 upper=3.14159 effort=23 velocity=30
- added joint RR_calf_joint: type revolute, parent rb_link2, child rb_link3, origin xyz=0.20711 0 0.0746 rpy=0 0 1.570796, axis 0 0 1, limit lower=-3.14159 upper=3.14159 effort=23 velocity=30
- added joint RR_foot_joint: type fixed, parent rb_link3, child rb_link4, origin xyz=0.22 0 0 rpy=3.1416 0 -1.5708, axis 0 0 0
- added joint RR_hip_joint: type revolute, parent body_link, child rb_link1, origin xyz=-0.20677 -0.06136 0.037786 rpy=-1.5708 0 1.5708, axis 0 0 1, limit lower=-3.14159 upper=3.14159 effort=23 velocity=30
- added joint RR_thigh_joint: type revolute, parent rb_link1, child rb_link2, origin xyz=-0.029301 1.3226E-05 0.06 rpy=-1.5708 0 1.5708, axis 0 0 1, limit lower=-3.14159 upper=3.14159 effort=23 velocity=30

Commit message: dog2挂载雷达和PC后的质量

File: source/robot_lab/data/Robots/atdog/dog2/urdf/dog2.urdf (robot description, URDF)
Before this commit: robot dog2, 17 links, 16 joints
Links:
- link base: mass 4.829 -> 5.791

Commit message: 调整ATDog2的URDF

File: source/robot_lab/data/Robots/atdog/dog2/urdf/dog2.urdf (robot description, URDF)
Before this commit: robot dog2, 17 links, 16 joints
Links:
- link base: mass 4.829 -> 5.236

Commit message: 调整ATDog2的URDF中关于关节限幅的参数

File: source/robot_lab/data/Robots/atdog/dog2/urdf/dog2.urdf (robot description, URDF)
Before this commit: robot dog2, 17 links, 16 joints
Joints:
- joint FL_calf_joint: limit lower=-3.14159 upper=3.14159 effort=23 velocity=30 -> lower=-1.0 upper=4.14159 effort=23 velocity=30
- joint FL_hip_joint: limit lower=-3.14159 upper=3.14159 effort=23 velocity=30 -> lower=-0.5 upper=1.0 effort=23 velocity=30
- joint FL_thigh_joint: limit lower=-3.14159 upper=3.14159 effort=23 velocity=30 -> lower=-1.57 upper=1.57 effort=23 velocity=30
- joint FR_calf_joint: limit lower=-3.14159 upper=3.14159 effort=23 velocity=30 -> lower=-4.14159 upper=1.0 effort=23 velocity=30
- joint FR_hip_joint: limit lower=-3.14159 upper=3.14159 effort=23 velocity=30 -> lower=-1.0 upper=0.5 effort=23 velocity=30
- joint FR_thigh_joint: limit lower=-3.14159 upper=3.14159 effort=23 velocity=30 -> lower=-1.57 upper=1.57 effort=23 velocity=30
- joint RL_calf_joint: limit lower=-3.14159 upper=3.14159 effort=23 velocity=30 -> lower=-1.0 upper=4.14159 effort=23 velocity=30
- joint RL_hip_joint: limit lower=-3.14159 upper=3.14159 effort=23 velocity=30 -> lower=-1.0 upper=0.5 effort=23 velocity=30
- joint RL_thigh_joint: limit lower=-3.14159 upper=3.14159 effort=23 velocity=30 -> lower=-1.57 upper=1.57 effort=23 velocity=30
- joint RR_calf_joint: limit lower=-3.14159 upper=3.14159 effort=23 velocity=30 -> lower=-4.14159 upper=1.0 effort=23 velocity=30
- joint RR_hip_joint: limit lower=-3.14159 upper=3.14159 effort=23 velocity=30 -> lower=-0.5 upper=1.0 effort=23 velocity=30
- joint RR_thigh_joint: limit lower=-3.14159 upper=3.14159 effort=23 velocity=30 -> lower=-1.57 upper=1.57 effort=23 velocity=30
