Commit message: 修正URDF关节限幅

File: source/robot_lab/data/Robots/atdog/dog2/urdf/dog2.urdf (robot description, URDF)
Before this commit: robot dog2, 17 links, 16 joints
Joints:
- joint FL_hip_joint: limit lower=-0.5 upper=1.0 effort=23 velocity=30 -> lower=-0.7 upper=1.5 effort=23 velocity=30
- joint FL_thigh_joint: limit lower=-1.57 upper=1.57 effort=23 velocity=30 -> lower=-2.4 upper=2.4 effort=23 velocity=30
- joint FR_hip_joint: limit lower=-1.0 upper=0.5 effort=23 velocity=30 -> lower=-1.5 upper=0.7 effort=23 velocity=30
- joint FR_thigh_joint: limit lower=-1.57 upper=1.57 effort=23 velocity=30 -> lower=-2.4 upper=2.4 effort=23 velocity=30
- joint RL_hip_joint: limit lower=-1.0 upper=0.5 effort=23 velocity=30 -> lower=-1.5 upper=0.7 effort=23 velocity=30
- joint RL_thigh_joint: limit lower=-1.57 upper=1.57 effort=23 velocity=30 -> lower=-2.4 upper=2.4 effort=23 velocity=30
- joint RR_hip_joint: limit lower=-0.5 upper=1.0 effort=23 velocity=30 -> lower=-0.7 upper=1.5 effort=23 velocity=30
- joint RR_thigh_joint: limit lower=-1.57 upper=1.57 effort=23 velocity=30 -> lower=-2.4 upper=2.4 effort=23 velocity=30

File: source/robot_lab/data/Robots/atdog/dog3/urdf/dog3.urdf (robot description, URDF)
Before this commit: robot dog3, 17 links, 16 joints
Joints:
- joint FL_hip_joint: limit lower=-0.5 upper=1.0 effort=30 velocity=30 -> lower=-0.7 upper=1.5 effort=30 velocity=30
- joint FL_thigh_joint: limit lower=-1.57 upper=1.57 effort=30 velocity=30 -> lower=-2.4 upper=2.4 effort=30 velocity=30
- joint FR_hip_joint: limit lower=-1.0 upper=0.5 effort=30 velocity=30 -> lower=-1.5 upper=0.7 effort=30 velocity=30
- joint FR_thigh_joint: limit lower=-1.57 upper=1.57 effort=30 velocity=30 -> lower=-2.4 upper=2.4 effort=30 velocity=30
- joint RL_hip_joint: limit lower=-1.0 upper=0.5 effort=30 velocity=30 -> lower=-1.5 upper=0.7 effort=30 velocity=30
- joint RL_thigh_joint: limit lower=-1.57 upper=1.57 effort=30 velocity=30 -> lower=-2.4 upper=2.4 effort=30 velocity=30
- joint RR_hip_joint: limit lower=-0.5 upper=1.0 effort=30 velocity=30 -> lower=-0.7 upper=1.5 effort=30 velocity=30
- joint RR_thigh_joint: limit lower=-1.57 upper=1.57 effort=30 velocity=30 -> lower=-2.4 upper=2.4 effort=30 velocity=30

File: source/robot_lab/data/Robots/atdog/dog3_arm/urdf/dog3_arm.urdf (robot description, URDF)
Before this commit: robot dog3_arm, 17 links, 16 joints
Joints:
- joint FL_calf_joint: limit lower=0 upper=0 effort=0 velocity=0 -> lower=-1.1 upper=1.1 effort=30 velocity=30
- joint FL_hip_joint: limit lower=0 upper=0 effort=0 velocity=0 -> lower=-0.7 upper=1.5 effort=30 velocity=30
- joint FL_thigh_joint: limit lower=0 upper=0 effort=0 velocity=0 -> lower=-2.4 upper=2.4 effort=30 velocity=30
- joint FR_calf_joint: limit lower=0 upper=0 effort=0 velocity=0 -> lower=-1.1 upper=1.1 effort=30 velocity=30
- joint FR_hip_joint: limit lower=0 upper=0 effort=0 velocity=0 -> lower=-1.5 upper=0.7 effort=30 velocity=30
- joint FR_thigh_joint: limit lower=0 upper=0 effort=0 velocity=0 -> lower=-2.4 upper=2.4 effort=30 velocity=30
- joint RL_calf_joint: limit lower=0 upper=0 effort=0 velocity=0 -> lower=-1.1 upper=1.1 effort=30 velocity=30
- joint RL_hip_joint: limit lower=0 upper=0 effort=0 velocity=0 -> lower=-1.5 upper=0.7 effort=30 velocity=30
- joint RL_thigh_joint: limit lower=0 upper=0 effort=0 velocity=0 -> lower=-2.4 upper=2.4 effort=30 velocity=30
- joint RR_calf_joint: limit lower=0 upper=0 effort=0 velocity=0 -> lower=-1.1 upper=1.1 effort=30 velocity=30
- joint RR_hip_joint: limit lower=0 upper=0 effort=0 velocity=0 -> lower=-0.7 upper=1.5 effort=30 velocity=30
- joint RR_thigh_joint: limit lower=0 upper=0 effort=0 velocity=0 -> lower=-2.4 upper=2.4 effort=30 velocity=30

Commit message: 最好的参数

File: source/robot_lab/data/Robots/atdog/dog2/urdf/dog2.urdf (robot description, URDF)
Before this commit: robot dog2, 17 links, 16 joints
Links:
- link base: mass 5.236 -> 6.236
