Commit message: 增加dog2的限高杆策略

File: source/robot_lab/data/Robots/atdog/dog2_arm/meshes/dog2_arm.urdf (robot description, URDF)
Before this commit: robot dog2_arm, 17 links, 16 joints
Links:
- link FL_calf: geometry collision mesh filename=lf_link3.stl; visual mesh filename=lf_link3.stl
- link FL_foot: geometry collision mesh filename=lf_link4.stl; visual mesh filename=lf_link4.stl
- link FL_hip: geometry collision mesh filename=lf_link1.stl; visual mesh filename=lf_link1.stl
- link FL_thigh: geometry collision mesh filename=lf_link2.stl; visual mesh filename=lf_link2.stl
- link FR_calf: geometry collision mesh filename=rf_link3.stl; visual mesh filename=rf_link3.stl
- link FR_foot: geometry collision mesh filename=rf_link4.stl; visual mesh filename=rf_link4.stl
- link FR_hip: geometry collision mesh filename=rf_link1.stl; visual mesh filename=rf_link1.stl
- link FR_thigh: geometry collision mesh filename=rf_link2.stl; visual mesh filename=rf_link2.stl
- link RL_calf: geometry collision mesh filename=lb_link3.stl; visual mesh filename=lb_link3.stl
- link RL_foot: geometry collision mesh filename=lb_link4.stl; visual mesh filename=lb_link4.stl
- link RL_hip: geometry collision mesh filename=lb_link1.stl; visual mesh filename=lb_link1.stl
- link RL_thigh: geometry collision mesh filename=lb_link2.stl; visual mesh filename=lb_link2.stl
- link RR_calf: geometry collision mesh filename=rb_link3.stl; visual mesh filename=rb_link3.stl
- link RR_foot: geometry collision mesh filename=rb_link4.stl; visual mesh filename=rb_link4.stl
- link RR_hip: geometry collision mesh filename=rb_link1.stl; visual mesh filename=rb_link1.stl
- link RR_thigh: geometry collision mesh filename=rb_link2.stl; visual mesh filename=rb_link2.stl
- link base: mass 6.33 -> 5.852583; geometry collision mesh filename=body_link.stl; visual mesh filename=body_link.stl

Commit message: 模型和训练策略更改

File: source/robot_lab/data/Robots/atdog/dog2_arm/meshes/dog2_arm.urdf (robot description, URDF)
Before this commit: robot dog2_arm, 17 links, 16 joints
Links:
- link base: mass 5.852583 -> 6.316865

File: source/robot_lab/data/Robots/atdog/dog2_arm/urdf/dog2_arm.urdf (robot description, URDF)
Before this commit: robot dog2_arm, 17 links, 16 joints
Links:
- link base: mass 5.852583 -> 6.316865

File: source/robot_lab/data/Robots/atdog/dog3/urdf/dog3.urdf (robot description, URDF)
Before this commit: robot dog3, 17 links, 16 joints
Links:
- link base: mass 5.314207 -> 5.814207
